File: hw/pcb/whisperbounce.kicad_sch (KiCad schematic)
At the start: 0 parts

Commit message: whisperbounce: Schematics
Signed-off-by: Dominik Sliwa <dominik@sliwa.io>
Parts:
- added FID1, FID2, FID3, FID4, FID5, FID6: Fiducial, symbol Mechanical:Fiducial
- added H1, H2, H3, H4: MountingHole_Pad, symbol Mechanical:MountingHole_Pad
Other:
- added sheet ETH Switch (eth_bridge.kicad_sch)
- added sheet USB ETH (usb_eth.kicad_sch)
- added sheet USB Hub (usb_hub.kicad_sch)
- added sheet USB-C (usb_c.kicad_sch)
- added sheet controller (controller.kicad_sch)
