File: hw/pcb/whisperbounce.kicad_sch (KiCad schematic)
At the start: 10 parts

Commit message: whisperbounce: assign footprints
Signed-off-by: Dominik Sliwa <dominik@sliwa.io>
Parts:
- FID1, FID2, FID3, FID4, FID5, FID6: footprint (none) -> Fiducial:Fiducial_0.75mm_Mask1.5mm
- H1, H2, H3, H4: footprint (none) -> MountingHole:MountingHole_3.2mm_M3_Pad_Via

Commit message: whisperbounce: pcb v1
Includes schematic and assigment tweaks

Signed-off-by: Dominik Sliwa <dominik@sliwa.io>
Changed lines of the file:
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@@
+    (stroke (width 0) (type solid) (color 0 0 0 0))
+  )
+  (wire (pts (xy 100.838 73.914) (xy 100.838 90.424))
+    (stroke (width 0) (type solid) (color 0 0 0 0))
+  )
+  (wire (pts (xy 100.838 90.424) (xy 103.124 90.424))
     (stroke (width 0) (type solid) (color 0 0 0 0))
   )
@@
   )
   (wire (pts (xy 101.854 88.392) (xy 103.124 88.392))
+    (stroke (width 0) (type solid) (color 0 0 0 0))
+  )
+  (wire (pts (xy 108.204 73.914) (xy 100.838 73.914))
     (stroke (width 0) (type solid) (color 0 0 0 0))
   )
@@
     )
     (property "Datasheet" "~" (id 3) (at 129.286 176.53 0)
+      (effects (font (size 1.27 1.27)) hide)
+    )
+  )
+  (symbol (lib_id "Graphic:Logo_Open_Hardware_Small") (at 163.322 167.894 0) (unit 1)
+    (in_bom yes) (on_board yes)
+    (property "Reference" "#LOGO1" (id 0) (at 163.322 160.909 0)
+      (effects (font (size 1.27 1.27)) hide)
+    )
+    (property "Value" "Logo_Open_Hardware_Small" (id 1) (at 163.322 173.609 0)
+      (effects (font (size 1.27 1.27)) hide)
+    )
+    (property "Footprint" "" (id 2) (at 163.322 167.894 0)
+      (effects (font (size 1.27 1.27)) hide)
+    )
+    (property "Datasheet" "~" (id 3) (at 163.322 167.894 0)
       (effects (font (size 1.27 1.27)) hide)
     )
@@
       (effects (font (size 1.27 1.27)) (justify right))
     )
-    (pin "LAN_USB3_RX+" input (at 108.204 44.704 180)
-      (effects (font (size 1.27 1.27)) (justify left))
-    )
-    (pin "LAN_USB3_RX-" input (at 108.204 46.482 180)
+    (pin "LAN_USB3_RX+" input (at 108.204 46.482 180)
+      (effects (font (size 1.27 1.27)) (justify left))
+    )
+    (pin "LAN_USB3_RX-" input (at 108.204 44.704 180)
       (effects (font (size 1.27 1.27)) (justify left))
     )
@@
   )
   (symbol_instances
+    (path "/42b6f9ba-1585-40fd-a18d-8137d0fab3bd"
+      (reference "#LOGO1") (unit 1) (value "Logo_Open_Hardware_Small") (footprint "")
+    )
     (path "/9101f65b-f4f4-42b0-a986-e7fa28fb955c"
       (reference "FID1") (unit 1) (value "Fiducial") (footprint "Fiducial:Fiducial_0.75mm_Mask1.5mm")
@@
       (reference "#PWR0101") (unit 1) (value "GND") (footprint "")
     )
-    (path "/af35eeca-deed-4d21-9f8e-d2051c9bf8b4/0abcf277-4e71-4211-91ce-ee819d069470"
-      (reference "#PWR0102") (unit 1) (value "GND") (footprint "")
-    )
     (path "/af35eeca-deed-4d21-9f8e-d2051c9bf8b4/ed460648-f5ca-4d35-ac56-db163e5424da"
       (reference "#PWR0103") (unit 1) (value "+3V3") (footprint "")
@@
       (reference "#PWR0124") (unit 1) (value "GND") (footprint "")
     )
-    (path "/af35eeca-deed-4d21-9f8e-d2051c9bf8b4/6e44014c-1c1f-45e8-af80-1ac67c61dd97"
-      (reference "#PWR0182") (unit 1) (value "GND") (footprint "")
-    )
     (path "/af35eeca-deed-4d21-9f8e-d2051c9bf8b4/2c099ee1-f9eb-476d-89e1-93af1213795a"
       (reference "C1") (unit 1) (value "0.1uF") (footprint "Capacitor_SMD:C_0402_1005Metric")
@@
       (reference "U4") (unit 1) (value "USB2422") (footprint "Package_DFN_QFN:QFN-24-1EP_4x4mm_P0.5mm_EP2.6x2.6mm")
     )
-    (path "/b5ba966d-72bb-41a5-98cc-df232cf77360/f8c73bea-1574-4554-866c-f73afcca7c87"
+    (path "/b5ba966d-72bb-41a5-98cc-df232cf77360/61f44af2-cb30-4448-ad39-b9e387e53e58"
       (reference "Y1") (unit 1) (value "24MHz") (footprint "Oscillator:Oscillator_SMD_Abracon_ASCO-4Pin_1.6x1.2mm")
     )
@@
       (reference "#PWR023") (unit 1) (value "GND") (footprint "")
     )
-    (path "/e152b1b6-46d9-4bd4-b218-e2d878c6a686/5172547b-fa7c-41e6-8f3b-169791737c5e"
-      (reference "#PWR026") (unit 1) (value "+3V3") (footprint "")
-    )
     (path "/e152b1b6-46d9-4bd4-b218-e2d878c6a686/bb75194e-7cfb-4099-855e-71f14ce9d01e"
       (reference "#PWR027") (unit 1) (value "GND") (footprint "")
@@
       (reference "#PWR031") (unit 1) (value "GND") (footprint "")
     )
-    (path "/e152b1b6-46d9-4bd4-b218-e2d878c6a686/831a72f1-1ba4-4b0e-a346-6df475ed3efd"
-      (reference "#PWR032") (unit 1) (value "+3V3") (footprint "")
-    )
     (path "/e152b1b6-46d9-4bd4-b218-e2d878c6a686/2c316e89-de0a-4f63-8f66-efe3f913c6e2"
       (reference "#PWR033") (unit 1) (value "GND") (footprint "")
@@
       (reference "#PWR035") (unit 1) (value "GND") (footprint "")
     )
-    (path "/e152b1b6-46d9-4bd4-b218-e2d878c6a686/db31810a-5550-4c68-9cc8-142f41d85f19"
-      (reference "#PWR036") (unit 1) (value "+3V3") (footprint "")
-    )
     (path "/e152b1b6-46d9-4bd4-b218-e2d878c6a686/6c7a900e-c3ea-4aeb-b0cc-43d46ebda374"
       (reference "#PWR037") (unit 1) (value "GND") (footprint "")
@@
       (reference "C30") (unit 1) (value "0.1uF") (footprint "Capacitor_SMD:C_0402_1005Metric")
     )
-    (path "/e152b1b6-46d9-4bd4-b218-e2d878c6a686/4efe810c-ae25-4e65-8476-6b482a999e10"
-      (reference "C31") (unit 1) (value "0.1uF") (footprint "Capacitor_SMD:C_0402_1005Metric")
-    )
     (path "/e152b1b6-46d9-4bd4-b218-e2d878c6a686/98d9a49c-9276-4a91-8361-4c3184eb2984"
       (reference "C32") (unit 1) (value "0.1uF") (footprint "Capacitor_SMD:C_0402_1005Metric")
@@
     )
     (path "/e152b1b6-46d9-4bd4-b218-e2d878c6a686/82c36f79-ffdf-4308-90e3-b0d1b1db412e"
-      (reference "L1") (unit 1) (value "3u3") (footprint "Inductor_SMD:L_Taiyo-Yuden_NR-40xx_HandSoldering")
+      (reference "L1") (unit 1) (value "3u3") (footprint "Inductor_SMD:L_Taiyo-Yuden_MD-2020")
     )
     (path "/e152b1b6-46d9-4bd4-b218-e2d878c6a686/3519bb58-290b-4a1a-af52-4ed247ceda0b"
@@
       (reference "#PWR055") (unit 1) (value "GND") (footprint "")
     )
+    (path "/3aba8689-8eba-492e-90d2-b70c101e638d/b4c1ca58-6038-487e-8d6e-b4543f6fc122"
+      (reference "#PWR092") (unit 1) (value "GND") (footprint "")
+    )
+    (path "/3aba8689-8eba-492e-90d2-b70c101e638d/6e80ede3-0c63-4db4-b342-a4283831dc2b"
+      (reference "#PWR093") (unit 1) (value "GND") (footprint "")
+    )
     (path "/3aba8689-8eba-492e-90d2-b70c101e638d/0a82fd8a-d788-4fce-942f-c6bb8930cb29"
       (reference "C44") (unit 1) (value "0.1uF") (footprint "Capacitor_SMD:C_0402_1005Metric")
@@
     )
     (path "/3aba8689-8eba-492e-90d2-b70c101e638d/48dd5629-bec9-47e2-8ec7-b57087ebd714"
-      (reference "SW2") (unit 1) (value "SW_Push") (footprint "Button_Switch_SMD:SW_SPST_B3U-3100P-B")
+      (reference "SW2") (unit 1) (value "SW_Push") (footprint "Button_Switch_SMD:SW_SPST_B3U-3000P")
     )
     (path "/3aba8689-8eba-492e-90d2-b70c101e638d/982bff2d-b6ae-4080-8de4-ae12850f5269"
       (reference "U7") (unit 1) (value "STM32F401CBUx") (footprint "Package_DFN_QFN:QFN-48-1EP_7x7mm_P0.5mm_EP5.6x5.6mm")
     )
-    (path "/3aba8689-8eba-492e-90d2-b70c101e638d/9f7f671e-edb1-4899-9747-f29b571b81c8"
-      (reference "Y2") (unit 1) (value "16MHz") (footprint "Oscillator:Oscillator_SMD_Abracon_ASCO-4Pin_1.6x1.2mm")
+    (path "/3aba8689-8eba-492e-90d2-b70c101e638d/4f0fac00-4a2b-41ff-bb59-d80baa188b86"
+      (reference "Y2") (unit 1) (value "24MHz") (footprint "Oscillator:Oscillator_SMD_Abracon_ASCO-4Pin_1.6x1.2mm")
     )
     (path "/6f3a1fa9-5359-4b3f-af72-6a88dfd458cc/47751da2-97d8-454c-b59e-56291e37487a"
