File: hw/pcb/controller.kicad_sch (KiCad schematic)
At the start: 19 parts, among them J2 Conn_01x10_MountingPin, SW1 SW_DP3T, SW2 SW_Push, U7 STM32F401CBUx, Y2 16MHz

Commit message: whisperbounce: assign footprints
Signed-off-by: Dominik Sliwa <dominik@sliwa.io>
Parts:
- removed SW1: SW_DP3T, symbol Switch:SW_DP3T
- added SW1: SW_SP3T, Button_Switch_SMD:SW_SP3T_PCM13, symbol Switch:SW_SP3T
- C44, C45, C46, C47, C48, C49, C50, C51, C52: footprint (none) -> Capacitor_SMD:C_0402_1005Metric
- J2: value Conn_01x10_MountingPin -> Debug connector; footprint (none) -> Connector_FFC-FPC:Hirose_FH12-10S-0.5SH_1x10-1MP_P0.50mm_Horizontal
- R17, R18, R19, R20, R21: footprint (none) -> Resistor_SMD:R_0402_1005Metric
- SW2: footprint (none) -> Button_Switch_SMD:SW_SPST_B3U-3100P-B
- Y2: footprint (none) -> Oscillator:Oscillator_SMD_Abracon_ASCO-4Pin_1.6x1.2mm
Connections:
- net +3V3: now also SW1.3
- net SW_A: now also SW1.1
- net SW_B: now also SW1.2
- net SW_C: now also SW1.4
- no-connect marks 21 -> 17
Changed lines of the file:
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@@
   (junction (at 150.114 139.446) (diameter 1.016) (color 0 0 0 0))
   (junction (at 152.654 139.446) (diameter 1.016) (color 0 0 0 0))
+  (no_connect (at 132.334 98.806))
+  (no_connect (at 132.334 88.646))
+  (no_connect (at 132.334 129.286))
+  (no_connect (at 132.334 124.206))
+  (no_connect (at 165.354 93.726))
+  (no_connect (at 132.334 121.666))
+  (no_connect (at 132.334 116.586))
+  (no_connect (at 132.334 131.826))
+  (no_connect (at 132.334 119.126))
+  (no_connect (at 236.22 83.82))
+  (no_connect (at 165.354 131.826))
   (no_connect (at 236.22 81.28))
-  (no_connect (at 236.22 83.82))
-  (no_connect (at 28.956 101.854))
-  (no_connect (at 39.116 99.314))
-  (no_connect (at 39.116 101.854))
-  (no_connect (at 39.116 104.394))
-  (no_connect (at 165.354 93.726))
   (no_connect (at 132.334 96.266))
-  (no_connect (at 132.334 98.806))
+  (no_connect (at 132.334 126.746))
   (no_connect (at 132.334 114.046))
-  (no_connect (at 132.334 116.586))
-  (no_connect (at 132.334 119.126))
-  (no_connect (at 132.334 121.666))
-  (no_connect (at 132.334 124.206))
-  (no_connect (at 132.334 126.746))
-  (no_connect (at 132.334 129.286))
-  (no_connect (at 132.334 131.826))
-  (no_connect (at 165.354 131.826))
+  (no_connect (at 132.334 91.186))
   (no_connect (at 132.334 86.106))
-  (no_connect (at 132.334 88.646))
-  (no_connect (at 132.334 91.186))
   (wire (pts (xy 23.622 26.67) (xy 23.622 22.352))
     (stroke (width 0) (type solid) (color 0 0 0 0))
@@
       (effects (font (size 1.27 1.27)) (justify right))
     )
-    (property "Footprint" "" (id 2) (at 50.292 84.328 0)
+    (property "Footprint" "Resistor_SMD:R_0402_1005Metric" (id 2) (at 50.292 84.328 0)
       (effects (font (size 1.27 1.27)) hide)
     )
@@
       (effects (font (size 1.27 1.27)) (justify right))
     )
-    (property "Footprint" "" (id 2) (at 50.292 86.868 0)
+    (property "Footprint" "Resistor_SMD:R_0402_1005Metric" (id 2) (at 50.292 86.868 0)
       (effects (font (size 1.27 1.27)) hide)
     )
@@
       (effects (font (size 1.27 1.27)) (justify right))
     )
-    (property "Footprint" "" (id 2) (at 50.292 89.408 0)
+    (property "Footprint" "Resistor_SMD:R_0402_1005Metric" (id 2) (at 50.292 89.408 0)
       (effects (font (size 1.27 1.27)) hide)
     )
@@
       (effects (font (size 1.27 1.27)) (justify right))
     )
-    (property "Footprint" "" (id 2) (at 111.506 61.976 0)
+    (property "Footprint" "Resistor_SMD:R_0402_1005Metric" (id 2) (at 111.506 61.976 0)
       (effects (font (size 1.27 1.27)) hide)
     )
@@
       (effects (font (size 1.27 1.27)) (justify right))
     )
-    (property "Footprint" "" (id 2) (at 119.126 101.346 0)
+    (property "Footprint" "Resistor_SMD:R_0402_1005Metric" (id 2) (at 119.126 101.346 0)
       (effects (font (size 1.27 1.27)) hide)
     )
@@
       (effects (font (size 1.27 1.27)) (justify left))
     )
-    (property "Footprint" "" (id 2) (at 33.02 32.512 0)
+    (property "Footprint" "Capacitor_SMD:C_0402_1005Metric" (id 2) (at 33.02 32.512 0)
       (effects (font (size 1.27 1.27)) hide)
     )
@@
       (effects (font (size 1.27 1.27)) (justify left))
     )
-    (property "Footprint" "" (id 2) (at 42.672 32.512 0)
+    (property "Footprint" "Capacitor_SMD:C_0402_1005Metric" (id 2) (at 42.672 32.512 0)
       (effects (font (size 1.27 1.27)) hide)
     )
@@
       (effects (font (size 1.27 1.27)) (justify left))
     )
-    (property "Footprint" "" (id 2) (at 52.07 32.512 0)
+    (property "Footprint" "Capacitor_SMD:C_0402_1005Metric" (id 2) (at 52.07 32.512 0)
       (effects (font (size 1.27 1.27)) hide)
     )
@@
       (effects (font (size 1.27 1.27)) (justify left))
     )
-    (property "Footprint" "" (id 2) (at 61.722 32.512 0)
+    (property "Footprint" "Capacitor_SMD:C_0402_1005Metric" (id 2) (at 61.722 32.512 0)
       (effects (font (size 1.27 1.27)) hide)
     )
@@
       (effects (font (size 1.27 1.27)) (justify left))
     )
-    (property "Footprint" "" (id 2) (at 71.12 32.512 0)
+    (property "Footprint" "Capacitor_SMD:C_0402_1005Metric" (id 2) (at 71.12 32.512 0)
       (effects (font (size 1.27 1.27)) hide)
     )
@@
     (property "Reference" "C49" (id 0) (at 107.569 73.406 90))
     (property "Value" "12pF" (id 1) (at 112.649 73.406 90))
-    (property "Footprint" "" (id 2) (at 109.474 75.946 0)
+    (property "Footprint" "Capacitor_SMD:C_0402_1005Metric" (id 2) (at 109.474 75.946 0)
       (effects (font (size 1.27 1.27)) hide)
     )
@@
     (property "Reference" "C50" (id 0) (at 107.569 86.741 90))
     (property "Value" "12pF" (id 1) (at 112.649 86.741 90))
-    (property "Footprint" "" (id 2) (at 109.474 83.566 0)
+    (property "Footprint" "Capacitor_SMD:C_0402_1005Metric" (id 2) (at 109.474 83.566 0)
       (effects (font (size 1.27 1.27)) hide)
     )
@@
       (effects (font (size 1.27 1.27)) (justify left))
     )
-    (property "Footprint" "" (id 2) (at 123.444 54.864 0)
+    (property "Footprint" "Capacitor_SMD:C_0402_1005Metric" (id 2) (at 123.444 54.864 0)
       (effects (font (size 1.27 1.27)) hide)
     )
@@
     (property "Reference" "C52" (id 0) (at 124.206 67.564 90))
     (property "Value" "4.7uF" (id 1) (at 130.556 67.564 90))
-    (property "Footprint" "" (id 2) (at 126.746 68.834 0)
+    (property "Footprint" "Capacitor_SMD:C_0402_1005Metric" (id 2) (at 126.746 68.834 0)
       (effects (font (size 1.27 1.27)) hide)
     )
@@
       (effects (font (size 1.27 1.27)) (justify right))
     )
-    (property "Footprint" "" (id 2) (at 117.856 79.756 0)
+    (property "Footprint" "Oscillator:Oscillator_SMD_Abracon_ASCO-4Pin_1.6x1.2mm" (id 2) (at 117.856 79.756 0)
       (effects (font (size 1.27 1.27)) hide)
     )
@@
     (property "Reference" "SW2" (id 0) (at 103.124 57.531 0))
     (property "Value" "SW_Push" (id 1) (at 103.124 60.071 0))
-    (property "Footprint" "" (id 2) (at 103.124 60.706 0)
+    (property "Footprint" "Button_Switch_SMD:SW_SPST_B3U-3100P-B" (id 2) (at 103.124 60.706 0)
       (effects (font (size 1.27 1.27)) hide)
     )
@@
     )
   )
-  (symbol (lib_id "Switch:SW_DP3T") (at 34.036 101.854 0) (unit 1)
-    (in_bom yes) (on_board yes)
-    (property "Reference" "SW1" (id 0) (at 34.036 93.599 0))
-    (property "Value" "SW_DP3T" (id 1) (at 34.036 96.139 0))
-    (property "Footprint" "" (id 2) (at 18.161 97.409 0)
-      (effects (font (size 1.27 1.27)) hide)
-    )
-    (property "Datasheet" "~" (id 3) (at 18.161 97.409 0)
-      (effects (font (size 1.27 1.27)) hide)
-    )
-  )
-  (symbol (lib_id "Switch:SW_DP3T") (at 35.306 86.868 0) (unit 2)
-    (in_bom yes) (on_board yes)
-    (property "Reference" "SW1" (id 0) (at 35.941 78.613 0))
-    (property "Value" "SW_DP3T" (id 1) (at 35.941 81.153 0))
-    (property "Footprint" "" (id 2) (at 19.431 82.423 0)
+  (symbol (lib_id "Switch:SW_SP3T") (at 35.306 86.868 0) (unit 1)
+    (in_bom yes) (on_board yes)
+    (property "Reference" "SW1" (id 0) (at 36.322 78.994 0))
+    (property "Value" "SW_SP3T" (id 1) (at 36.322 81.534 0))
+    (property "Footprint" "Button_Switch_SMD:SW_SP3T_PCM13" (id 2) (at 19.431 82.423 0)
       (effects (font (size 1.27 1.27)) hide)
     )
@@
       (effects (font (size 1.27 1.27)) (justify left))
     )
-    (property "Value" "Conn_01x10_MountingPin" (id 1) (at 244.221 74.93 0)
-      (effects (font (size 1.27 1.27)) (justify left))
-    )
-    (property "Footprint" "" (id 2) (at 241.3 71.12 0)
-      (effects (font (size 1.27 1.27)) hide)
-    )
+    (property "Value" "Debug connector" (id 1) (at 244.221 74.93 0)
+      (effects (font (size 1.27 1.27)) (justify left))
+    )
+    (property "Footprint" "Connector_FFC-FPC:Hirose_FH12-10S-0.5SH_1x10-1MP_P0.50mm_Horizontal" (id 2) (at 241.3 71.12 0)
+      (effects (font (size 1.27 1.27)) hide)
+    )

Commit message: whisperbounce: pcb v1
Includes schematic and assigment tweaks

Signed-off-by: Dominik Sliwa <dominik@sliwa.io>
Parts:
- removed Y2: 16MHz, Oscillator:Oscillator_SMD_Abracon_ASCO-4Pin_1.6x1.2mm, symbol Device:Crystal_GND23_Small
- added Y2: 24MHz, Oscillator:Oscillator_SMD_Abracon_ASCO-4Pin_1.6x1.2mm, symbol Device:Crystal_GND24_Small
- SW2: footprint Button_Switch_SMD:SW_SPST_B3U-3100P-B -> Button_Switch_SMD:SW_SPST_B3U-3000P
Connections:
- net GND: now also Y2.2, Y2.4
- net at C50.2, U7.6 (PH1): now also Y2.1
- net at C49.2, U7.5 (PH0): now also Y2.3
Changed lines of the file:
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@@
   (junction (at 150.114 139.446) (diameter 1.016) (color 0 0 0 0))
   (junction (at 152.654 139.446) (diameter 1.016) (color 0 0 0 0))
-  (no_connect (at 132.334 98.806))
+  (no_connect (at 132.334 86.106))
+  (no_connect (at 132.334 116.586))
   (no_connect (at 132.334 88.646))
   (no_connect (at 132.334 129.286))
+  (no_connect (at 132.334 119.126))
+  (no_connect (at 165.354 131.826))
+  (no_connect (at 132.334 96.266))
+  (no_connect (at 132.334 98.806))
+  (no_connect (at 132.334 126.746))
+  (no_connect (at 132.334 121.666))
+  (no_connect (at 236.22 81.28))
+  (no_connect (at 132.334 114.046))
+  (no_connect (at 132.334 131.826))
+  (no_connect (at 165.354 93.726))
   (no_connect (at 132.334 124.206))
-  (no_connect (at 165.354 93.726))
-  (no_connect (at 132.334 121.666))
-  (no_connect (at 132.334 116.586))
-  (no_connect (at 132.334 131.826))
-  (no_connect (at 132.334 119.126))
+  (no_connect (at 132.334 91.186))
   (no_connect (at 236.22 83.82))
-  (no_connect (at 165.354 131.826))
-  (no_connect (at 236.22 81.28))
-  (no_connect (at 132.334 96.266))
-  (no_connect (at 132.334 126.746))
-  (no_connect (at 132.334 114.046))
-  (no_connect (at 132.334 91.186))
-  (no_connect (at 132.334 86.106))
   (wire (pts (xy 23.622 26.67) (xy 23.622 22.352))
     (stroke (width 0) (type solid) (color 0 0 0 0))
@@
     (stroke (width 0) (type solid) (color 0 0 0 0))
   )
+  (wire (pts (xy 114.046 79.756) (xy 115.316 79.756))
+    (stroke (width 0) (type solid) (color 0 0 0 0))
+  )
   (wire (pts (xy 114.046 101.346) (xy 116.586 101.346))
     (stroke (width 0) (type solid) (color 0 0 0 0))
@@
   )
   (wire (pts (xy 117.856 83.566) (xy 129.286 83.566))
+    (stroke (width 0) (type solid) (color 0 0 0 0))
+  )
+  (wire (pts (xy 121.666 79.756) (xy 120.396 79.756))
     (stroke (width 0) (type solid) (color 0 0 0 0))
   )
@@
     )
   )
+  (symbol (lib_id "power:GND") (at 114.046 79.756 270) (unit 1)
+    (in_bom yes) (on_board yes)
+    (property "Reference" "#PWR092" (id 0) (at 107.696 79.756 0)
+      (effects (font (size 1.27 1.27)) hide)
+    )
+    (property "Value" "GND" (id 1) (at 110.871 79.121 90)
+      (effects (font (size 1.27 1.27)) (justify right))
+    )
+    (property "Footprint" "" (id 2) (at 114.046 79.756 0)
+      (effects (font (size 1.27 1.27)) hide)
+    )
+    (property "Datasheet" "" (id 3) (at 114.046 79.756 0)
+      (effects (font (size 1.27 1.27)) hide)
+    )
+  )
   (symbol (lib_id "power:GND") (at 114.046 101.346 270) (unit 1)
     (in_bom yes) (on_board yes)
@@
     )
     (property "Datasheet" "" (id 3) (at 114.046 101.346 0)
+      (effects (font (size 1.27 1.27)) hide)
+    )
+  )
+  (symbol (lib_id "power:GND") (at 121.666 79.756 90) (unit 1)
+    (in_bom yes) (on_board yes)
+    (property "Reference" "#PWR093" (id 0) (at 128.016 79.756 0)
+      (effects (font (size 1.27 1.27)) hide)
+    )
+    (property "Value" "GND" (id 1) (at 124.841 80.391 90)
+      (effects (font (size 1.27 1.27)) (justify right))
+    )
+    (property "Footprint" "" (id 2) (at 121.666 79.756 0)
+      (effects (font (size 1.27 1.27)) hide)
+    )
+    (property "Datasheet" "" (id 3) (at 121.666 79.756 0)
       (effects (font (size 1.27 1.27)) hide)
     )
@@
     )
   )
-  (symbol (lib_id "Device:Crystal_GND23_Small") (at 117.856 79.756 90) (unit 1)
-    (in_bom yes) (on_board yes)
-    (property "Reference" "Y2" (id 0) (at 122.301 77.851 90)
-      (effects (font (size 1.27 1.27)) (justify right))
-    )
-    (property "Value" "16MHz" (id 1) (at 122.301 80.391 90)
+  (symbol (lib_id "Device:Crystal_GND24_Small") (at 117.856 79.756 90) (unit 1)
+    (in_bom yes) (on_board yes)
+    (property "Reference" "Y2" (id 0) (at 120.65 77.47 90)
+      (effects (font (size 1.27 1.27)) (justify right))
+    )
+    (property "Value" "24MHz" (id 1) (at 120.65 82.296 90)
       (effects (font (size 1.27 1.27)) (justify right))
     )
@@
     (property "Reference" "SW2" (id 0) (at 103.124 57.531 0))
     (property "Value" "SW_Push" (id 1) (at 103.124 60.071 0))
-    (property "Footprint" "Button_Switch_SMD:SW_SPST_B3U-3100P-B" (id 2) (at 103.124 60.706 0)
-      (effects (font (size 1.27 1.27)) hide)
-    )
+    (property "Footprint" "Button_Switch_SMD:SW_SPST_B3U-3000P" (id 2) (at 103.124 60.706 0)
+      (effects (font (size 1.27 1.27)) hide)
+    )
