File: hw/pcb/eth_bridge.kicad_sch (KiCad schematic)
At the start: 58 parts, among them J3 JK0654219, J4 JK0654219, U8 MUN12AD01-SH, U9 KSZ9893RNX, X1 ASE-xxxMHz

Commit message: whisperbounce: assign footprints
Signed-off-by: Dominik Sliwa <dominik@sliwa.io>
Parts:
- FB10, FB5, FB6, FB7, FB8, FB9: footprint (none) -> Resistor_SMD:R_0603_1608Metric
- U9: footprint Package_DFN_QFN:QFN-64-1EP_8x8mm_P0.4mm_EP6.5x6.5mm -> Package_DFN_QFN:QFN-64-1EP_8x8mm_P0.4mm_EP6.5x6.5mm_ThermalVias
- X1: footprint Oscillator:Oscillator_SMD_Abracon_ASE-4Pin_3.2x2.5mm -> Oscillator:Oscillator_SMD_Abracon_ASCO-4Pin_1.6x1.2mm
Changed lines of the file:
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@@
   (junction (at 229.87 133.35) (diameter 1.016) (color 0 0 0 0))
   (no_connect (at 118.11 135.255))
+  (no_connect (at 118.11 114.935))
   (no_connect (at 118.11 89.535))
   (no_connect (at 118.11 69.215))
   (no_connect (at 59.69 29.845))
   (no_connect (at 39.37 29.845))
-  (no_connect (at 118.11 114.935))
   (wire (pts (xy 17.78 151.13) (xy 17.78 147.32))
     (stroke (width 0) (type solid) (color 0 0 0 0))
@@
     (property "Reference" "FB5" (id 0) (at 24.003 144.78 90))
     (property "Value" "220" (id 1) (at 24.003 147.32 90))
-    (property "Footprint" "" (id 2) (at 23.495 152.908 90)
+    (property "Footprint" "Resistor_SMD:R_0603_1608Metric" (id 2) (at 23.495 152.908 90)
       (effects (font (size 1.27 1.27)) hide)
     )
@@
     (property "Reference" "FB6" (id 0) (at 25.273 52.07 90))
     (property "Value" "220" (id 1) (at 25.273 54.61 90))
-    (property "Footprint" "" (id 2) (at 24.765 60.198 90)
+    (property "Footprint" "Resistor_SMD:R_0603_1608Metric" (id 2) (at 24.765 60.198 90)
       (effects (font (size 1.27 1.27)) hide)
     )
@@
     (property "Reference" "FB7" (id 0) (at 25.273 81.28 90))
     (property "Value" "220" (id 1) (at 25.273 83.82 90))
-    (property "Footprint" "" (id 2) (at 24.765 89.408 90)
+    (property "Footprint" "Resistor_SMD:R_0603_1608Metric" (id 2) (at 24.765 89.408 90)
       (effects (font (size 1.27 1.27)) hide)
     )
@@
     (property "Reference" "FB8" (id 0) (at 25.273 110.49 90))
     (property "Value" "220" (id 1) (at 25.273 113.03 90))
-    (property "Footprint" "" (id 2) (at 24.765 118.618 90)
+    (property "Footprint" "Resistor_SMD:R_0603_1608Metric" (id 2) (at 24.765 118.618 90)
       (effects (font (size 1.27 1.27)) hide)
     )
@@
     (property "Reference" "FB9" (id 0) (at 255.397 77.724 90))
     (property "Value" "220" (id 1) (at 255.397 80.264 90))
-    (property "Footprint" "" (id 2) (at 254.635 86.868 90)
+    (property "Footprint" "Resistor_SMD:R_0603_1608Metric" (id 2) (at 254.635 86.868 90)
       (effects (font (size 1.27 1.27)) hide)
     )
@@
     (property "Reference" "FB10" (id 0) (at 255.143 149.86 90))
     (property "Value" "220" (id 1) (at 255.143 152.4 90))
-    (property "Footprint" "" (id 2) (at 254.635 157.988 90)
+    (property "Footprint" "Resistor_SMD:R_0603_1608Metric" (id 2) (at 254.635 157.988 90)
       (effects (font (size 1.27 1.27)) hide)
     )
@@
       (effects (font (size 1.27 1.27)) (justify left))
     )
-    (property "Footprint" "Oscillator:Oscillator_SMD_Abracon_ASE-4Pin_3.2x2.5mm" (id 2) (at 203.2 43.18 0)
+    (property "Footprint" "Oscillator:Oscillator_SMD_Abracon_ASCO-4Pin_1.6x1.2mm" (id 2) (at 203.2 43.18 0)
       (effects (font (size 1.27 1.27)) hide)
     )
@@
     (property "Reference" "U9" (id 0) (at 121.92 139.065 0))
     (property "Value" "KSZ9893RNX" (id 1) (at 185.674 139.065 0))
-    (property "Footprint" "Package_DFN_QFN:QFN-64-1EP_8x8mm_P0.4mm_EP6.5x6.5mm" (id 2) (at 156.21 53.975 0)
-      (effects (font (size 1.27 1.27)) hide)
-    )
+    (property "Footprint" "Package_DFN_QFN:QFN-64-1EP_8x8mm_P0.4mm_EP6.5x6.5mm_ThermalVias" (id 2) (at 156.21 53.975 0)
+      (effects (font (size 1.27 1.27)) hide)
+    )
